File: PCB/Key_PN532/aic_key_pn532.kicad_sch (KiCad schematic)
At the start: 33 parts, among them J1 PN532, SW1 SKRR_4pin, SW10 SKRR_4pin, SW11 SKRR_4pin, SW12 SKRR_4pin, SW2 SKRR_4pin, SW3 SKRR_4pin, SW4 SKRR_4pin, SW5 SKRR_4pin, SW6 SKRR_4pin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

Commit message: WS2812C-2020 option for AIC Key PN532
Parts:
- added D13, D14, D15, D16, D17, D18: WS2812B_Unified, aic_pico:WS2812C-2020, symbol aic_pico:WS2812B_Unified
Connections:
- net +5V: now also D13.V (VDD), D14.V (VDD), D15.V (VDD), D16.V (VDD), D17.V (VDD), D18.V (VDD)
- net GND: now also D13.G (VSS), D14.G (VSS), D15.G (VSS), D16.G (VSS), D17.G (VSS), D18.G (VSS)
- net L1: now reaches D1.I (In), R1.1
- net L1: now also D13.I (In)
- net L2: now reaches D1.O (Out), D2.I (In)
- net L2: now also D13.O (Out), D14.I (In)
- net L3: now reaches D2.O (Out), D3.I (In)
- net L3: now also D14.O (Out), D15.I (In)
- net L4: now reaches D3.O (Out), D4.I (In)
- net L4: now also D15.O (Out), D16.I (In)
- net L5: now reaches D4.O (Out), D5.I (In)
- net L5: now also D16.O (Out), D17.I (In)
- net L6: now reaches D5.O (Out), D6.I (In)
- net L6: now also D17.O (Out), D18.I (In)
- no-connect marks 12 -> 13
