File: PCB/Key_PN5180/aic_pico_pn5180.kicad_pcb (KiCad board)
At the start: 2 copper layers, 50 x 50 mm, 34 parts, among them J1 Conn_01x02_Female, J2 PN5180, SW1 SKRR_4pin, SW10 SKRR_4pin, SW11 SKRR_4pin, SW12 SKRR_4pin, SW2 SKRR_4pin, SW3 SKRR_4pin, SW4 SKRR_4pin, SW5 SKRR_4pin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

Commit message: Power filtering for PN5180 on AIC Key
Parts:
- added C1: 0.1uF, Capacitor_SMD:C_0603_1608Metric, B.Cu at (121.6, 95.4)
- added C2: 10uF, Capacitor_SMD:C_0603_1608Metric, B.Cu at (119.3, 131.2)
- added L1: 100nH, Inductor_SMD:L_0805_2012Metric, B.Cu at (119.8, 95.1)
Connections:
- J2 pad 1: +5V -> Net-(J2-5V)
Routing:
- net Net-(J2-5V): track 0.00 -> 49.3 mm
- net +5V: track 159.7 -> 113.8 mm
- net GND: track 335.8 -> 337.5 mm
Other:
- board text added: "AIC Key v1.3"
- board text removed: "AIC Key v1.2"

Commit message: L1 to 1206 and power from VBUS
Parts:
- L1: footprint Inductor_SMD:L_0805_2012Metric -> Inductor_SMD:L_1206_3216Metric
- moved C1 2.58 mm to (119.0, 95.4)
- moved L1 1.37 mm to (121.1, 94.6)
Connections:
- L1 pad 1: +5V -> Net-(U1-VBUS)
- U1 pad 40: unconnected-(U1-VBUS-Pad40) -> Net-(U1-VBUS)
Routing:
- net Net-(U1-VBUS): track 0.00 -> 7.29 mm
- net +5V: track 113.8 -> 106.8 mm
- net GND: track 337.5 -> 340.1 mm
- net Net-(J2-5V): track 49.3 -> 48.8 mm
Other:
- board text added: "AIC Key v1.31"
- board text removed: "AIC Key v1.3"
