File: PCB/Key/aic_key.kicad_sch (KiCad schematic)
At the start: 37 parts, among them J1 Conn_01x02_Female, J2 PN5180, SW1 SKRR_4pin, SW10 SKRR_4pin, SW11 SKRR_4pin, SW12 SKRR_4pin, SW2 SKRR_4pin, SW3 SKRR_4pin, SW4 SKRR_4pin, SW5 SKRR_4pin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

Commit message: Hybrid AIC Key PCB and AIC touch RGB back to 1204
Parts:
- removed C2: 10uF, Capacitor_SMD:C_0603_1608Metric, symbol Device:C
- removed L1: 100nH, Inductor_SMD:L_1206_3216Metric, symbol Device:L
- added J3: PN532, aic_pico:pn532_conn, symbol aic_pico:PN532
Connections:
- net +3V3: now also J3.2 (VCC)
- net +5V: now also C1.1, J2.1 (5V)
- net GND: now also J3.1 (GND)
- net at U1.26 (GPIO20): now also J3.3 (SDA)
- net at U1.27 (GPIO21): now also J3.4 (SCL)
- no-connect marks 11 -> 9
