File: PCB/Key/aic_key.kicad_sch (KiCad schematic)
At the start: 36 parts, among them J1 Conn_01x02_Female, J2 PN5180, J3 PN532, SW1 SKRR_4pin, SW10 SKRR_4pin, SW11 SKRR_4pin, SW12 SKRR_4pin, SW2 SKRR_4pin, SW3 SKRR_4pin, SW4 SKRR_4pin, SW5 SKRR_4pin, SW6 SKRR_4pin, SW7 SKRR_4pin, SW8 SKRR_4pin, SW9 SKRR_4pin, U1 Pico_Trim

Commit message: AIC Key PCB v1.51 (minor finetune)
Parts:
- removed C1: 0.1uF, Capacitor_SMD:C_0603_1608Metric, symbol Device:C
- removed R1: 10, Resistor_SMD:R_0603_1608Metric, symbol Device:R_Small
Connections:
- net at D1.I (In): now also U1.16 (GPIO12)
